File: FARA_KEYBOARD/FARA_KEYBOARD.kicad_sch (KiCad schematic)
At the start: 20 parts, among them J1 Conn_01x07_Pin, J2 Conn_01x20, J3 Conn_01x20, J4 Conn_01x04, J5 Conn_01x03, J6 Conn_01x03, J7 Conn_01x03, J8 Conn_01x03, J9 Conn_01x03, SW1 SW_Push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

Commit message: v0.4 circuit is ready
Parts:
- added BZ1: Buzzer, Connector_PinHeader_2.54mm:PinHeader_1x02_P2.54mm_Vertical, symbol Device:Buzzer
- added J10, J13: Conn_01x02, Connector_PinSocket_2.54mm:PinSocket_1x02_P2.54mm_Vertical, symbol Connector_Generic:Conn_01x02
- added J11, J12: Screw_Terminal_01x02, Connector_PinSocket_2.54mm:PinSocket_1x02_P2.54mm_Vertical, symbol Connector:Screw_Terminal_01x02
- added Q1, Q2: AO3400A, Package_TO_SOT_SMD:SOT-23, symbol Transistor_FET:AO3400A
- added R5, R6: 0, Resistor_SMD:R_0201_0603Metric, symbol Device:R
Connections:
- net STRIP4 is gone; now on net STRIP3: J3.20 (Pin_20), J9.2 (Pin_2), U1.20 (GP15)
- net +3V3: now also R6.2
- net +5V: now also R5.2
- net GND: now also BZ1.2 (+), J10.2 (Pin_2), J13.2 (Pin_2), Q1.2 (S), Q2.2 (S)
- net STRIP1: now also J3.17 (Pin_17), J7.2 (Pin_2), U1.17 (GP13); no longer J3.16 (Pin_16), J6.2 (Pin_2), U1.16 (GP12)
- net STRIP2: now also J3.19 (Pin_19), J8.2 (Pin_2), U1.19 (GP14); no longer J3.17 (Pin_17), J7.2 (Pin_2), U1.17 (GP13)
- net STRIP3: no longer J3.19 (Pin_19), J8.2 (Pin_2), U1.19 (GP14)
- net buzzer: now reaches J2.14 (Pin_14), U1.27 (GP21)
- net buzzer: now also BZ1.1 (-)
- net lasers: now reaches J2.20 (Pin_20), U1.21 (GP16/MISO)
- net lasers: now also Q2.1 (G)
- net LEDS: now reaches J3.5 (Pin_5), U1.5 (GP3)
- net LEDS: now also J13.1 (Pin_1), Q1.1 (G)
- new net: J11.2 (Pin_2), J12.2 (Pin_2), Q2.3 (D)
- new net: J10.1 (Pin_1), Q1.3 (D)
- new net STRIP0: J3.16 (Pin_16), J6.2 (Pin_2), U1.16 (GP12)
- new net V_lasers: J11.1 (Pin_1), J12.1 (Pin_1), R5.1, R6.1

Commit message: v0.5 draft PCB was routed
Parts:
- added Q3: AO3400A, Package_TO_SOT_SMD:SOT-23, symbol Transistor_FET:AO3400A
- added R7: 0, Resistor_SMD:R_0805_2012Metric_Pad1.20x1.40mm_HandSolder, symbol Device:R
- R3, R4, R5, R6: footprint Resistor_SMD:R_0201_0603Metric -> Resistor_SMD:R_0402_1005Metric_Pad0.72x0.64mm_HandSolder
- U1: footprint Shield_Emergent:Raspberry Pi Pico -> myLib8:Raspberry Pi Pico
Connections:
- net +3V3: no longer R1.1, R2.1
- net +5V: now also BZ1.1 (-), R7.1
- net GND: now also Q3.2 (S); no longer BZ1.2 (+)
- net VPP: now also R7.2
- net buzzer: now also Q3.1 (G); no longer BZ1.1 (-)
- net V_I2C: now reaches J4.4 (Pin_4), R3.1, R4.1
- net V_I2C: now also R1.1, R2.1
- new net: BZ1.2 (+), Q3.3 (D)
Other:
- moved on the sheet: BZ1, J5

Commit message: v0.6 seems 2B ready
Parts:
- added D1: PMEG3010CEH, Diode_SMD:D_SOD-123F, symbol Diode:PMEG3010CEH
Connections:
- net +5V: now also D1.1 (K)
- net at BZ1.2 (+), Q3.3 (D): now also D1.2 (A)
Other:
- moved on the sheet: BZ1, SW1, SW2

Commit message: v0.7 form was corrected
Parts:
- added J14: Conn_01x02, Connector_PinSocket_2.54mm:PinSocket_1x02_P2.54mm_Vertical, symbol Connector_Generic:Conn_01x02
Connections:
- net GND: now also J14.2 (Pin_2)
- net FLT_I/O: now reaches J2.17 (Pin_17), U1.24 (GP18/SCK)
- net FLT_I/O: now also J14.1 (Pin_1)
Other:
- moved on the sheet: BZ1, D1, J10, J11, J12, J13, J2, J3, J4, Q1, Q2, Q3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
